Commit message: '24.12.19'

File: body.urdf (robot description, URDF)
Before this commit: robot robot, 3 links, 2 joints
Links:
- removed link L_Leg
- removed link R_Leg
- added link LLeg, mass 1; collision box size=1 1 1; visual box size=1 1 1
- added link RLeg, mass 1; collision box size=1 1 1; visual box size=1 1 1
Joints:
- removed joint Torso_L_Leg
- removed joint Torso_R_Leg
- added joint Torso_LLeg: type fixed, parent Torso, child LLeg, origin xyz=-0.5 0 1.5 rpy=0 0 0, axis 0 1 0, limit lower=-3.14159 upper=3.14159 effort=0.0 velocity=0.0
- added joint Torso_RLeg: type fixed, parent Torso, child RLeg, origin xyz=0.5 0 1.5 rpy=0 0 0, axis 0 1 0, limit lower=-3.14159 upper=3.14159 effort=0.0 velocity=0.0

Commit message: '24.12.19'

File: body.urdf (robot description, URDF)
Before this commit: robot robot, 3 links, 2 joints
Joints:
- joint Torso_LLeg: origin xyz=-0.5 0 1.5 rpy=0 0 0 -> xyz=-0.5 0 1 rpy=0 0 0; type fixed -> revolute
- joint Torso_RLeg: origin xyz=0.5 0 1.5 rpy=0 0 0 -> xyz=0.5 0 1 rpy=0 0 0; type fixed -> revolute
